Commit message: Added new robot

File: envs/assets/robotV2/Robot_description/urdf/Robot.urdf (robot description, URDF)
Before this commit: robot Robot, 13 links, 12 joints
Links:
- removed link left_ankle_link_1
- removed link left_calf_link_1
- removed link left_foot_link_1
- removed link left_hip_pitch_link_1
- removed link left_hip_yaw_link_1
- removed link left_thigh_link_1
- removed link right_ankle_link_1
- removed link right_calf_link_1
- removed link right_foot_link_1
- removed link right_hip_pitch_link_1
- removed link right_hip_yaw_link_1
- removed link right_thigh_link_1
- added link l_ankle_link_1, mass 0.021339; collision mesh filename=package://Robot_description/meshes/l_ankle_link_1.stl scale=0.001 0.001 0.001; visual mesh filename=package://Robot_description/meshes/l_ankle_link_1.stl scale=0.001 0.001 0.001
- added link l_calf_link_1, mass 0.10503; collision mesh filename=package://Robot_description/meshes/l_calf_link_1.stl scale=0.001 0.001 0.001; visual mesh filename=package://Robot_description/meshes/l_calf_link_1.stl scale=0.001 0.001 0.001
- added link l_foot_link_1, mass 0.096795; collision mesh filename=package://Robot_description/meshes/l_foot_link_1.stl scale=0.001 0.001 0.001; visual mesh filename=package://Robot_description/meshes/l_foot_link_1.stl scale=0.001 0.001 0.001
- added link l_hip_lower_link_1, mass 0.021339; collision mesh filename=package://Robot_description/meshes/l_hip_lower_link_1.stl scale=0.001 0.001 0.001; visual mesh filename=package://Robot_description/meshes/l_hip_lower_link_1.stl scale=0.001 0.001 0.001
- added link l_hip_upper_link_1, mass 0.100649; collision mesh filename=package://Robot_description/meshes/l_hip_upper_link_1.stl scale=0.001 0.001 0.001; visual mesh filename=package://Robot_description/meshes/l_hip_upper_link_1.stl scale=0.001 0.001 0.001
- added link l_thigh_link_1, mass 0.168697; collision mesh filename=package://Robot_description/meshes/l_thigh_link_1.stl scale=0.001 0.001 0.001; visual mesh filename=package://Robot_description/meshes/l_thigh_link_1.stl scale=0.001 0.001 0.001
- added link r_ankle_link_1, mass 0.021339; collision mesh filename=package://Robot_description/meshes/r_ankle_link_1.stl scale=0.001 0.001 0.001; visual mesh filename=package://Robot_description/meshes/r_ankle_link_1.stl scale=0.001 0.001 0.001
- added link r_calf_link_1, mass 0.10503; collision mesh filename=package://Robot_description/meshes/r_calf_link_1.stl scale=0.001 0.001 0.001; visual mesh filename=package://Robot_description/meshes/r_calf_link_1.stl scale=0.001 0.001 0.001
- added link r_foot_link_1, mass 0.096795; collision mesh filename=package://Robot_description/meshes/r_foot_link_1.stl scale=0.001 0.001 0.001; visual mesh filename=package://Robot_description/meshes/r_foot_link_1.stl scale=0.001 0.001 0.001
- added link r_hip_lower_link_1, mass 0.021339; collision mesh filename=package://Robot_description/meshes/r_hip_lower_link_1.stl scale=0.001 0.001 0.001; visual mesh filename=package://Robot_description/meshes/r_hip_lower_link_1.stl scale=0.001 0.001 0.001
- added link r_hip_upper_link_1, mass 0.100649; collision mesh filename=package://Robot_description/meshes/r_hip_upper_link_1.stl scale=0.001 0.001 0.001; visual mesh filename=package://Robot_description/meshes/r_hip_upper_link_1.stl scale=0.001 0.001 0.001
- added link r_thigh_link_1, mass 0.168697; collision mesh filename=package://Robot_description/meshes/r_thigh_link_1.stl scale=0.001 0.001 0.001; visual mesh filename=package://Robot_description/meshes/r_thigh_link_1.stl scale=0.001 0.001 0.001
- link base_link: mass 0.685004957374252 -> 0.622478
Joints:
- removed joint left_ankle_pitch
- removed joint left_ankle_roll
- removed joint left_hip_pitch
- removed joint left_hip_roll
- removed joint left_hip_yaw
- removed joint left_knee
- removed joint right_ankle_pitch
- removed joint right_ankle_roll
- removed joint right_hip_pitch
- removed joint right_hip_roll
- removed joint right_hip_yaw
- removed joint right_knee
- added joint l_ankle_pitch_joint: type revolute, parent l_ankle_link_1, child l_foot_link_1, origin xyz=-0.018625 -0.020625 -0.0339 rpy=0 0 0, axis -0.0 1.0 -0.0, limit lower=-0.610865 upper=1.48353 effort=100 velocity=100
- added joint l_ankle_roll_joint: type revolute, parent l_calf_link_1, child l_ankle_link_1, origin xyz=0.018625 0.019101 -0.072184 rpy=0 0 0, axis 1.0 -0.0 0.0, limit lower=-1.396263 upper=1.396263 effort=100 velocity=100
- added joint l_hip_pitch_joint: type revolute, parent l_hip_lower_link_1, child l_thigh_link_1, origin xyz=-0.018625 -0.020625 -0.0339 rpy=0 0 0, axis 0.0 1.0 0.0, limit lower=-1.570796 upper=1.570796 effort=100 velocity=100
- added joint l_hip_roll_joint: type revolute, parent l_hip_upper_link_1, child l_hip_lower_link_1, origin xyz=0.0191 0.030829 -0.040776 rpy=0 0 0, axis 1.0 -0.0 0.0, limit lower=-0.436332 upper=1.570796 effort=100 velocity=100
- added joint l_hip_yaw: type revolute, parent base_link, child l_hip_upper_link_1, origin xyz=-0.00159 0.021672 -0.00015 rpy=0 0 0, axis 0.0 0.0 1.0, limit lower=-0.785398 upper=0.785398 effort=100 velocity=100
- added joint l_knee_joint: type revolute, parent l_thigh_link_1, child l_calf_link_1, origin xyz=0.0 0.002 -0.072052 rpy=0 0 0, axis -0.0 -1.0 -0.0, limit lower=-2.094395 upper=2.094395 effort=100 velocity=100
- added joint r_ankle_pitch_joint: type revolute, parent r_ankle_link_1, child r_foot_link_1, origin xyz=-0.018625 0.020625 -0.0339 rpy=0 0 0, axis 0.0 1.0 0.0, limit lower=-0.610865 upper=1.48353 effort=100 velocity=100
- added joint r_ankle_roll_joint: type revolute, parent r_calf_link_1, child r_ankle_link_1, origin xyz=0.018625 -0.019101 -0.072184 rpy=0 0 0, axis -1.0 -0.0 -0.0, limit lower=-1.396263 upper=1.396263 effort=100 velocity=100
- added joint r_hip_pitch_joint: type revolute, parent r_hip_lower_link_1, child r_thigh_link_1, origin xyz=-0.018625 0.020625 -0.0339 rpy=0 0 0, axis -0.0 1.0 -0.0, limit lower=-1.570796 upper=1.570796 effort=100 velocity=100
- added joint r_hip_roll_joint: type revolute, parent r_hip_upper_link_1, child r_hip_lower_link_1, origin xyz=0.0191 -0.030829 -0.040776 rpy=0 0 0, axis -1.0 -0.0 -0.0, limit lower=-0.436332 upper=1.570796 effort=100 velocity=100
- added joint r_hip_yaw: type revolute, parent base_link, child r_hip_upper_link_1, origin xyz=-0.00159 -0.021672 -0.00015 rpy=0 0 0, axis -0.0 -0.0 -1.0, limit lower=-0.785398 upper=0.785398 effort=100 velocity=100
- added joint r_knee_joint: type revolute, parent r_thigh_link_1, child r_calf_link_1, origin xyz=0.0 -0.002 -0.072052 rpy=0 0 0, axis 0.0 -1.0 0.0, limit lower=-2.094395 upper=2.094395 effort=100 velocity=100

Commit message: New body

File: envs/assets/robotV2/Robot_description/urdf/Robot.urdf (robot description, URDF)
Before this commit: robot Robot, 13 links, 12 joints
Links:
- added link imu_link, mass 0.0
- link base_link: mass 0.622478 -> 0.633299
Joints:
- added joint imu_joint: type fixed, parent base_link, child imu_link, origin xyz=-0.023673 0.0 0.025133 rpy=0 0 0
